File: rpi_pico_kit/rpi_pico_kit.kicad_sch (KiCad schematic)
At the start: 2 parts, among them SW1 SW_Push_Dual, U1 Pico

Commit message: added leds for uart, little changes
Parts:
- added C? (x2): 100n, symbol Device:C
- added D? (x2): LL4148, Diode_SMD:D_MiniMELF, symbol Diode:LL4148
- added D? (x2): LED, LED_SMD:LED_1206_3216Metric_Pad1.42x1.75mm_HandSolder, symbol Device:LED
- added J?: Conn_01x03_Male, symbol Connector:Conn_01x03_Male
- added Q? (x2): BC807, Package_TO_SOT_SMD:SOT-23, symbol Transistor_BJT:BC807
- added R? (x2): 100R, Resistor_SMD:R_0805_2012Metric_Pad1.20x1.40mm_HandSolder, symbol Device:R
- added R? (x4): 1k, Resistor_SMD:R_0805_2012Metric_Pad1.20x1.40mm_HandSolder, symbol Device:R
- added R? (x2): 10k, Resistor_SMD:R_0805_2012Metric_Pad1.20x1.40mm_HandSolder, symbol Device:R
Connections:
- net +3V3: now also C?.2, C?.2, Q?.3 (C), Q?.3 (C)
- net GND: now also J?.2 (Pin_2), R?.2, R?.2
- net UART0_RX: now also R?.1, R?.2
- net UART0_TX: now also R?.1, R?.2
- new net: D?.1 (K), R?.2 (x2)
- new net: C?.1, D?.2 (A), R?.1 (x2)
- new net: D?.1 (K), R?.1 (x2)
- new net: D?.2 (A), Q?.2 (E) (x2)
- new net: Q?.1 (B), R?.2 (x2)
- new net: J?.1 (Pin_1), R?.1
- new net: J?.3 (Pin_3), R?.1
