File: rpi_pico_kit/audio.kicad_sch (KiCad schematic)
At the start: 36 parts, among them J10 AudioJack-CUI-SJ-3523-SMT, J11 AudioJack-CUI-SJ-3523-SMT, Q7 BSS138, U7 NC7WZ16P6X, U8 PCM5101A, U9 TLV70033_SOT23-5

Commit message: added some footprints
Parts:
- C26, C28, C30, C32, C34, C35, C36: footprint (none) -> Capacitor_SMD:C_0805_2012Metric_Pad1.18x1.45mm_HandSolder
Changed lines of the file:
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@@
       (effects (font (size 1.27 1.27)) (justify right))
     )
-    (property "Footprint" "" (id 2) (at 96.8248 111.76 0)
+    (property "Footprint" "Capacitor_SMD:C_0805_2012Metric_Pad1.18x1.45mm_HandSolder" (id 2) (at 96.8248 111.76 0)
       (effects (font (size 1.27 1.27)) hide)
     )
@@
       (effects (font (size 1.27 1.27)) (justify right))
     )
-    (property "Footprint" "" (id 2) (at 86.6648 157.48 0)
+    (property "Footprint" "Capacitor_SMD:C_0805_2012Metric_Pad1.18x1.45mm_HandSolder" (id 2) (at 86.6648 157.48 0)
       (effects (font (size 1.27 1.27)) hide)
     )
@@
       (effects (font (size 1.27 1.27)) (justify right))
     )
-    (property "Footprint" "" (id 2) (at 87.9348 139.7 0)
+    (property "Footprint" "Capacitor_SMD:C_0805_2012Metric_Pad1.18x1.45mm_HandSolder" (id 2) (at 87.9348 139.7 0)
       (effects (font (size 1.27 1.27)) hide)
     )
@@
       (effects (font (size 1.27 1.27)))
     )
-    (property "Footprint" "" (id 2) (at 110.49 32.0548 0)
+    (property "Footprint" "Capacitor_SMD:C_0805_2012Metric_Pad1.18x1.45mm_HandSolder" (id 2) (at 110.49 32.0548 0)
       (effects (font (size 1.27 1.27)) hide)
     )
@@
       (effects (font (size 1.27 1.27)) (justify right))
     )
-    (property "Footprint" "" (id 2) (at 57.4548 111.76 0)
+    (property "Footprint" "Capacitor_SMD:C_0805_2012Metric_Pad1.18x1.45mm_HandSolder" (id 2) (at 57.4548 111.76 0)
       (effects (font (size 1.27 1.27)) hide)
     )
@@
       (effects (font (size 1.27 1.27)) (justify right))
     )
-    (property "Footprint" "" (id 2) (at 123.4948 111.76 0)
+    (property "Footprint" "Capacitor_SMD:C_0805_2012Metric_Pad1.18x1.45mm_HandSolder" (id 2) (at 123.4948 111.76 0)
       (effects (font (size 1.27 1.27)) hide)
     )
@@
       (effects (font (size 1.27 1.27)))
     )
-    (property "Footprint" "" (id 2) (at 110.49 59.9948 0)
-      (effects (font (size 1.27 1.27)) hide)
-    )
+    (property "Footprint" "Capacitor_SMD:C_0805_2012Metric_Pad1.18x1.45mm_HandSolder" (id 2) (at 110.49 59.9948 0)
+      (effects (font (size 1.27 1.27)) hide)
+    )

Commit message: added some footprints and MPNs
Parts:
- BZ1: footprint (none) -> Buzzer_Beeper:Buzzer_12x9.5RM7.6; Manufacturer Part Number (none) -> LA216001; Supplier (none) -> Laskakit; Supplier Part URL (none) -> https://www.laskakit.cz/pasivni-bzucak--5v
- J10, J11: Manufacturer Part Number (none) -> SJ-3523-SMT-TR; Supplier (none) -> Digikey; Supplier Part URL (none) -> https://www.digikey.cz/en/products/detail/cui-devices/SJ-35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
Changed lines of the file:
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@@
+      (effects (font (size 1.27 1.27)) hide)
+    )
+    (property "Manufacturer Part Number" "SJ-3523-SMT-TR" (id 5) (at 133.35 49.53 0)
+      (effects (font (size 1.27 1.27)) hide)
+    )
+    (property "Supplier" "Digikey" (id 6) (at 133.35 49.53 0)
+      (effects (font (size 1.27 1.27)) hide)
+    )
+    (property "Supplier Part URL" "https://www.digikey.cz/en/products/detail/cui-devices/SJ-3523-SMT-TR/281297" (id 7) (at 133.35 49.53 0)
       (effects (font (size 1.27 1.27)) hide)
     )
@@
     )
     (property "Datasheet" "" (id 3) (at 144.78 134.62 0)
+      (effects (font (size 1.27 1.27)) hide)
+    )
+    (property "Manufacturer Part Number" "SJ-3523-SMT-TR" (id 6) (at 144.78 134.62 0)
+      (effects (font (size 1.27 1.27)) hide)
+    )
+    (property "Supplier" "Digikey" (id 7) (at 144.78 134.62 0)
+      (effects (font (size 1.27 1.27)) hide)
+    )
+    (property "Supplier Part URL" "https://www.digikey.cz/en/products/detail/cui-devices/SJ-3523-SMT-TR/281297" (id 8) (at 144.78 134.62 0)
       (effects (font (size 1.27 1.27)) hide)
     )
@@
       (effects (font (size 1.27 1.27)) (justify left))
     )
-    (property "Footprint" "" (id 2) (at 244.475 100.33 90)
+    (property "Footprint" "Buzzer_Beeper:Buzzer_12x9.5RM7.6" (id 2) (at 244.475 100.33 90)
       (effects (font (size 1.27 1.27)) hide)
     )
@@
       (effects (font (size 1.27 1.27)) hide)
     )
+    (property "Manufacturer Part Number" "LA216001" (id 4) (at 245.11 102.87 0)
+      (effects (font (size 1.27 1.27)) hide)
+    )
+    (property "Supplier" "Laskakit" (id 5) (at 245.11 102.87 0)
+      (effects (font (size 1.27 1.27)) hide)
+    )
+    (property "Supplier Part URL" "https://www.laskakit.cz/pasivni-bzucak--5v" (id 6) (at 245.11 102.87 0)
+      (effects (font (size 1.27 1.27)) hide)
+    )

Commit message: added MPNs for capacitors
Parts:
- C24, C25, C27, C29, C31, C33, C37: Manufacturer Part Number (none) -> C0805C104M3RAC7800; Supplier (none) -> Digikey; Supplier Part URL (none) -> https://www.digikey.cz/en/products/detail/kemet/C0805C104M3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
- C26, C28: Manufacturer Part Number (none) -> CL21A476MRYNNNE; Supplier (none) -> Digikey; Supplier Part URL (none) -> https://www.digikey.cz/en/products/detail/samsung-electro-m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
- C30, C32, C34: Manufacturer Part Number (none) -> CL21A106KOQNNNG; Supplier (none) -> Digikey; Supplier Part URL (none) -> https://www.digikey.cz/en/products/detail/samsung-electro-m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
- C35, C36: Manufacturer Part Number (none) -> C0805C225Z4VAC7800; Supplier (none) -> Digikey; Supplier Part URL (none) -> https://www.digikey.cz/en/products/detail/kemet/C0805C225Z4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
- C38, C39: Manufacturer Part Number (none) -> C0805C222K5RAC7800; Supplier (none) -> Digikey; Supplier Part URL (none) -> https://www.digikey.cz/en/products/detail/kemet/C0805C222K5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
- C40, C41: Manufacturer Part Number (none) -> C0805C105Z4VAC7800; Supplier (none) -> Digikey; Supplier Part URL (none) -> https://www.digikey.cz/en/products/detail/kemet/C0805C105Z4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
Changed lines of the file:
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@@
+      (effects (font (size 1.27 1.27)) hide)
+    )
+    (property "Manufacturer Part Number" "C0805C104M3RAC7800" (id 4) (at 99.06 161.29 0)
+      (effects (font (size 1.27 1.27)) hide)
+    )
+    (property "Supplier" "Digikey" (id 5) (at 99.06 161.29 0)
+      (effects (font (size 1.27 1.27)) hide)
+    )
+    (property "Supplier Part URL" "https://www.digikey.cz/en/products/detail/kemet/C0805C104M3RAC7800/2211748" (id 6) (at 99.06 161.29 0)
       (effects (font (size 1.27 1.27)) hide)
     )
@@
       (effects (font (size 1.27 1.27)) hide)
     )
+    (property "Manufacturer Part Number" "C0805C104M3RAC7800" (id 4) (at 113.03 115.57 0)
+      (effects (font (size 1.27 1.27)) hide)
+    )
+    (property "Supplier" "Digikey" (id 5) (at 113.03 115.57 0)
+      (effects (font (size 1.27 1.27)) hide)
+    )
+    (property "Supplier Part URL" "https://www.digikey.cz/en/products/detail/kemet/C0805C104M3RAC7800/2211748" (id 6) (at 113.03 115.57 0)
+      (effects (font (size 1.27 1.27)) hide)
+    )
     (pin "1")
     (pin "2")
@@
       (effects (font (size 1.27 1.27)) hide)
     )
+    (property "Manufacturer Part Number" "C0805C104M3RAC7800" (id 4) (at 86.36 115.57 0)
+      (effects (font (size 1.27 1.27)) hide)
+    )
+    (property "Supplier" "Digikey" (id 5) (at 86.36 115.57 0)
+      (effects (font (size 1.27 1.27)) hide)
+    )
+    (property "Supplier Part URL" "https://www.digikey.cz/en/products/detail/kemet/C0805C104M3RAC7800/2211748" (id 6) (at 86.36 115.57 0)
+      (effects (font (size 1.27 1.27)) hide)
+    )
     (pin "1")
     (pin "2")
@@
     )
     (property "Datasheet" "~" (id 3) (at 243.84 64.77 0)
+      (effects (font (size 1.27 1.27)) hide)
+    )
+    (property "Manufacturer Part Number" "C0805C105Z4VAC7800" (id 4) (at 243.84 64.77 0)
+      (effects (font (size 1.27 1.27)) hide)
+    )
+    (property "Supplier" "Digikey" (id 5) (at 243.84 64.77 0)
+      (effects (font (size 1.27 1.27)) hide)
+    )
+    (property "Supplier Part URL" "https://www.digikey.cz/en/products/detail/kemet/C0805C105Z4VAC7800/2211782" (id 6) (at 243.84 64.77 0)
       (effects (font (size 1.27 1.27)) hide)
     )
@@
       (effects (font (size 1.27 1.27)) hide)
     )
+    (property "Manufacturer Part Number" "C0805C222K5RAC7800" (id 4) (at 113.03 142.24 0)
+      (effects (font (size 1.27 1.27)) hide)
+    )
+    (property "Supplier" "Digikey" (id 5) (at 113.03 142.24 0)
+      (effects (font (size 1.27 1.27)) hide)
+    )
+    (property "Supplier Part URL" "https://www.digikey.cz/en/products/detail/kemet/C0805C222K5RAC7800/411150" (id 6) (at 113.03 142.24 0)
+      (effects (font (size 1.27 1.27)) hide)
+    )
     (pin "1")
     (pin "2")
@@
       (effects (font (size 1.27 1.27)) hide)
     )
+    (property "Manufacturer Part Number" "CL21A106KOQNNNG" (id 4) (at 97.79 115.57 0)
+      (effects (font (size 1.27 1.27)) hide)
+    )
+    (property "Supplier" "Digikey" (id 5) (at 97.79 115.57 0)
+      (effects (font (size 1.27 1.27)) hide)
+    )
+    (property "Supplier Part URL" "https://www.digikey.cz/en/products/detail/samsung-electro-mechanics/CL21A106KOQNNNG/3894417" (id 6) (at 97.79 115.57 0)
+      (effects (font (size 1.27 1.27)) hide)
+    )
     (pin "1")
     (pin "2")
@@
       (effects (font (size 1.27 1.27)) hide)
     )
+    (property "Manufacturer Part Number" "C0805C225Z4VAC7800" (id 4) (at 87.63 161.29 0)
+      (effects (font (size 1.27 1.27)) hide)
+    )
+    (property "Supplier" "Digikey" (id 5) (at 87.63 161.29 0)
+      (effects (font (size 1.27 1.27)) hide)
+    )
+    (property "Supplier Part URL" "https://www.digikey.cz/en/products/detail/kemet/C0805C225Z4VAC7800/417855" (id 6) (at 87.63 161.29 0)
+      (effects (font (size 1.27 1.27)) hide)
+    )
     (pin "1")
     (pin "2")
@@
       (effects (font (size 1.27 1.27)) hide)
     )
+    (property "Manufacturer Part Number" "C0805C225Z4VAC7800" (id 4) (at 88.9 143.51 0)
+      (effects (font (size 1.27 1.27)) hide)
+    )
+    (property "Supplier" "Digikey" (id 5) (at 88.9 143.51 0)
+      (effects (font (size 1.27 1.27)) hide)
+    )
+    (property "Supplier Part URL" "https://www.digikey.cz/en/products/detail/kemet/C0805C225Z4VAC7800/417855" (id 6) (at 88.9 143.51 0)
+      (effects (font (size 1.27 1.27)) hide)
+    )
     (pin "1")
     (pin "2")
@@
       (effects (font (size 1.27 1.27)) hide)
     )
+    (property "Manufacturer Part Number" "CL21A476MRYNNNE" (id 4) (at 106.68 33.02 0)
+      (effects (font (size 1.27 1.27)) hide)
+    )
+    (property "Supplier" "Digikey" (id 5) (at 106.68 33.02 0)
+      (effects (font (size 1.27 1.27)) hide)
+    )
+    (property "Supplier Part URL" "https://www.digikey.cz/en/products/detail/samsung-electro-mechanics/CL21A476MRYNNNE/3888577" (id 6) (at 106.68 33.02 0)
+      (effects (font (size 1.27 1.27)) hide)
+    )
     (pin "1")
     (pin "2")
@@
       (effects (font (size 1.27 1.27)) hide)
     )
+    (property "Manufacturer Part Number" "C0805C222K5RAC7800" (id 4) (at 124.46 142.24 0)
+      (effects (font (size 1.27 1.27)) hide)
+    )
+    (property "Supplier" "Digikey" (id 5) (at 124.46 142.24 0)
+      (effects (font (size 1.27 1.27)) hide)
+    )
+    (property "Supplier Part URL" "https://www.digikey.cz/en/products/detail/kemet/C0805C222K5RAC7800/411150" (id 6) (at 124.46 142.24 0)
+      (effects (font (size 1.27 1.27)) hide)
+    )
     (pin "1")
     (pin "2")
@@
       (effects (font (size 1.27 1.27)) hide)
     )
+    (property "Manufacturer Part Number" "CL21A106KOQNNNG" (id 4) (at 58.42 115.57 0)
+      (effects (font (size 1.27 1.27)) hide)
+    )
+    (property "Supplier" "Digikey" (id 5) (at 58.42 115.57 0)
+      (effects (font (size 1.27 1.27)) hide)
+    )
+    (property "Supplier Part URL" "https://www.digikey.cz/en/products/detail/samsung-electro-mechanics/CL21A106KOQNNNG/3894417" (id 6) (at 58.42 115.57 0)
+      (effects (font (size 1.27 1.27)) hide)
+    )
     (pin "1")
     (pin "2")
@@
       (effects (font (size 1.27 1.27)) hide)
     )
+    (property "Manufacturer Part Number" "C0805C104M3RAC7800" (id 4) (at 46.99 115.57 0)
+      (effects (font (size 1.27 1.27)) hide)
+    )
+    (property "Supplier" "Digikey" (id 5) (at 46.99 115.57 0)
+      (effects (font (size 1.27 1.27)) hide)
+    )
+    (property "Supplier Part URL" "https://www.digikey.cz/en/products/detail/kemet/C0805C104M3RAC7800/2211748" (id 6) (at 46.99 115.57 0)
+      (effects (font (size 1.27 1.27)) hide)
+    )
     (pin "1")
     (pin "2")
@@
     )
     (property "Datasheet" "~" (id 3) (at 210.82 64.77 0)
+      (effects (font (size 1.27 1.27)) hide)
+    )
+    (property "Manufacturer Part Number" "C0805C105Z4VAC7800" (id 4) (at 210.82 64.77 0)
+      (effects (font (size 1.27 1.27)) hide)
+    )
+    (property "Supplier" "Digikey" (id 5) (at 210.82 64.77 0)
+      (effects (font (size 1.27 1.27)) hide)
+    )
+    (property "Supplier Part URL" "https://www.digikey.cz/en/products/detail/kemet/C0805C105Z4VAC7800/2211782" (id 6) (at 210.82 64.77 0)
       (effects (font (size 1.27 1.27)) hide)
     )
@@
     )
     (property "Datasheet" "~" (id 3) (at 88.9 39.37 0)
+      (effects (font (size 1.27 1.27)) hide)
+    )
+    (property "Manufacturer Part Number" "C0805C104M3RAC7800" (id 4) (at 88.9 39.37 0)
+      (effects (font (size 1.27 1.27)) hide)
+    )
+    (property "Supplier" "Digikey" (id 5) (at 88.9 39.37 0)
+      (effects (font (size 1.27 1.27)) hide)
+    )
+    (property "Supplier Part URL" "https://www.digikey.cz/en/products/detail/kemet/C0805C104M3RAC7800/2211748" (id 6) (at 88.9 39.37 0)
       (effects (font (size 1.27 1.27)) hide)
     )
@@
       (effects (font (size 1.27 1.27)) hide)
     )
+    (property "Manufacturer Part Number" "CL21A106KOQNNNG" (id 4) (at 124.46 115.57 0)
+      (effects (font (size 1.27 1.27)) hide)
+    )
+    (property "Supplier" "Digikey" (id 5) (at 124.46 115.57 0)
+      (effects (font (size 1.27 1.27)) hide)
+    )
+    (property "Supplier Part URL" "https://www.digikey.cz/en/products/detail/samsung-electro-mechanics/CL21A106KOQNNNG/3894417" (id 6) (at 124.46 115.57 0)
+      (effects (font (size 1.27 1.27)) hide)
+    )
     (pin "1")
     (pin "2")
@@
       (effects (font (size 1.27 1.27)) hide)
     )
+    (property "Manufacturer Part Number" "C0805C104M3RAC7800" (id 4) (at 67.31 52.07 0)
+      (effects (font (size 1.27 1.27)) hide)
+    )
+    (property "Supplier" "Digikey" (id 5) (at 67.31 52.07 0)
+      (effects (font (size 1.27 1.27)) hide)
+    )
+    (property "Supplier Part URL" "https://www.digikey.cz/en/products/detail/kemet/C0805C104M3RAC7800/2211748" (id 6) (at 67.31 52.07 0)
+      (effects (font (size 1.27 1.27)) hide)
+    )
     (pin "1")
     (pin "2")
@@
     )
     (property "Datasheet" "~" (id 3) (at 88.9 67.31 0)
+      (effects (font (size 1.27 1.27)) hide)
+    )
+    (property "Manufacturer Part Number" "C0805C104M3RAC7800" (id 4) (at 88.9 67.31 0)
+      (effects (font (size 1.27 1.27)) hide)
+    )
+    (property "Supplier" "Digikey" (id 5) (at 88.9 67.31 0)
+      (effects (font (size 1.27 1.27)) hide)
+    )
+    (property "Supplier Part URL" "https://www.digikey.cz/en/products/detail/kemet/C0805C104M3RAC7800/2211748" (id 6) (at 88.9 67.31 0)
       (effects (font (size 1.27 1.27)) hide)
     )
@@
       (effects (font (size 1.27 1.27)) hide)
     )
+    (property "Manufacturer Part Number" "CL21A476MRYNNNE" (id 4) (at 106.68 60.96 0)
+      (effects (font (size 1.27 1.27)) hide)
+    )
+    (property "Supplier" "Digikey" (id 5) (at 106.68 60.96 0)
+      (effects (font (size 1.27 1.27)) hide)
+    )
+    (property "Supplier Part URL" "https://www.digikey.cz/en/products/detail/samsung-electro-mechanics/CL21A476MRYNNNE/3888577" (id 6) (at 106.68 60.96 0)
+      (effects (font (size 1.27 1.27)) hide)
+    )
