File: rpi_pico_kit/spi_devices.kicad_sch (KiCad schematic)
At the start: 20 parts, among them J6 Conn_01x08_Male, J7 Conn_01x08_Male, J8 Conn_01x08_Male, J9 Micro_SD_Card_Det, SW10 SW_Push, SW7 SW_Push, SW8 SW_Push, SW9 SW_Push, U7 MCP23S08-xSO

Commit message: added missing footprints
Parts:
- RN4, RN5, RN6, RN7: footprint (none) -> Resistor_SMD:R_Array_Convex_4x1206
Changed lines of the file:
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@@
       (effects (font (size 1.27 1.27)) (justify right))
     )
-    (property "Footprint" "" (id 2) (at 116.332 73.66 90)
+    (property "Footprint" "Resistor_SMD:R_Array_Convex_4x1206" (id 2) (at 116.332 73.66 90)
       (effects (font (size 1.27 1.27)) hide)
     )
@@
       (effects (font (size 1.27 1.27)) (justify right))
     )
-    (property "Footprint" "" (id 2) (at 123.19 57.658 90)
+    (property "Footprint" "Resistor_SMD:R_Array_Convex_4x1206" (id 2) (at 123.19 57.658 90)
       (effects (font (size 1.27 1.27)) hide)
     )
@@
       (effects (font (size 1.27 1.27)) (justify right))
     )
-    (property "Footprint" "" (id 2) (at 135.382 73.66 90)
+    (property "Footprint" "Resistor_SMD:R_Array_Convex_4x1206" (id 2) (at 135.382 73.66 90)
       (effects (font (size 1.27 1.27)) hide)
     )
@@
       (effects (font (size 1.27 1.27)) (justify right))
     )
-    (property "Footprint" "" (id 2) (at 89.662 73.66 90)
+    (property "Footprint" "Resistor_SMD:R_Array_Convex_4x1206" (id 2) (at 89.662 73.66 90)
       (effects (font (size 1.27 1.27)) hide)
     )
@@
       (effects (font (size 1.27 1.27)) (justify right))
     )
-    (property "Footprint" "" (id 2) (at 111.76 123.698 90)
+    (property "Footprint" "Resistor_SMD:R_Array_Convex_4x1206" (id 2) (at 111.76 123.698 90)
       (effects (font (size 1.27 1.27)) hide)
     )
@@
       (effects (font (size 1.27 1.27)) (justify right))
     )
-    (property "Footprint" "" (id 2) (at 123.19 62.738 90)
+    (property "Footprint" "Resistor_SMD:R_Array_Convex_4x1206" (id 2) (at 123.19 62.738 90)
       (effects (font (size 1.27 1.27)) hide)
     )
@@
       (effects (font (size 1.27 1.27)) (justify right))
     )
-    (property "Footprint" "" (id 2) (at 111.76 128.778 90)
+    (property "Footprint" "Resistor_SMD:R_Array_Convex_4x1206" (id 2) (at 111.76 128.778 90)
       (effects (font (size 1.27 1.27)) hide)
     )
@@
       (effects (font (size 1.27 1.27)) (justify right))
     )
-    (property "Footprint" "" (id 2) (at 173.482 73.66 90)
+    (property "Footprint" "Resistor_SMD:R_Array_Convex_4x1206" (id 2) (at 173.482 73.66 90)
       (effects (font (size 1.27 1.27)) hide)
     )
@@
       (effects (font (size 1.27 1.27)) (justify right))
     )
-    (property "Footprint" "" (id 2) (at 123.19 60.198 90)
+    (property "Footprint" "Resistor_SMD:R_Array_Convex_4x1206" (id 2) (at 123.19 60.198 90)
       (effects (font (size 1.27 1.27)) hide)
     )
@@
       (effects (font (size 1.27 1.27)) (justify right))
     )
-    (property "Footprint" "" (id 2) (at 111.76 138.938 90)
+    (property "Footprint" "Resistor_SMD:R_Array_Convex_4x1206" (id 2) (at 111.76 138.938 90)
       (effects (font (size 1.27 1.27)) hide)
     )
@@
       (effects (font (size 1.27 1.27)) (justify right))
     )
-    (property "Footprint" "" (id 2) (at 148.082 73.66 90)
+    (property "Footprint" "Resistor_SMD:R_Array_Convex_4x1206" (id 2) (at 148.082 73.66 90)
       (effects (font (size 1.27 1.27)) hide)
     )
@@
       (effects (font (size 1.27 1.27)) (justify right))
     )
-    (property "Footprint" "" (id 2) (at 98.552 73.66 90)
+    (property "Footprint" "Resistor_SMD:R_Array_Convex_4x1206" (id 2) (at 98.552 73.66 90)
       (effects (font (size 1.27 1.27)) hide)
     )
@@
       (effects (font (size 1.27 1.27)) (justify right))
     )
-    (property "Footprint" "" (id 2) (at 107.442 73.66 90)
+    (property "Footprint" "Resistor_SMD:R_Array_Convex_4x1206" (id 2) (at 107.442 73.66 90)
       (effects (font (size 1.27 1.27)) hide)
     )
@@
       (effects (font (size 1.27 1.27)) (justify right))
     )
-    (property "Footprint" "" (id 2) (at 111.76 133.858 90)
+    (property "Footprint" "Resistor_SMD:R_Array_Convex_4x1206" (id 2) (at 111.76 133.858 90)
       (effects (font (size 1.27 1.27)) hide)
     )
@@
       (effects (font (size 1.27 1.27)) (justify right))
     )
-    (property "Footprint" "" (id 2) (at 123.19 65.278 90)
+    (property "Footprint" "Resistor_SMD:R_Array_Convex_4x1206" (id 2) (at 123.19 65.278 90)
       (effects (font (size 1.27 1.27)) hide)
     )
@@
       (effects (font (size 1.27 1.27)) (justify right))
     )
-    (property "Footprint" "" (id 2) (at 160.782 73.66 90)
-      (effects (font (size 1.27 1.27)) hide)
-    )
+    (property "Footprint" "Resistor_SMD:R_Array_Convex_4x1206" (id 2) (at 160.782 73.66 90)
+      (effects (font (size 1.27 1.27)) hide)
+    )
