File: rpi_pico_kit/basic_ui.kicad_sch (KiCad schematic)
At the start: 30 parts, among them Q3 DMN63D8L-7, Q4 DMN63D8L-7, Q5 DMN63D8L-7, Q6 DMN63D8L-7, SW2 RotaryEncoder_Switch, SW3 SW_Push, SW4 SW_Push, SW5 SW_Push, SW6 SW_Push, U6 74HC14

Commit message: changed footprints from 0805 to 0603
Parts:
- C23: footprint Capacitor_SMD:C_0805_2012Metric_Pad1.18x1.45mm_HandSolder -> Capacitor_SMD:C_0603_1608Metric_Pad1.08x0.95mm_HandSolder; Supplier Part URL https://www.digikey.cz/en/products/detail/kemet/C0805C104M3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 -> (none)
- R37, R38, R39, R40, R46, R47, R49, R51: footprint Resistor_SMD:R_0805_2012Metric_Pad1.20x1.40mm_HandSolder -> Resistor_SMD:R_0603_1608Metric_Pad0.98x0.95mm_HandSolder; Supplier Part URL https://www.digikey.cz/en/products/detail/yageo/RC0805FR-07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 -> (none)
Changed lines of the file:
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@@
       (effects (font (size 1.27 1.27)))
     )
-    (property "Footprint" "Resistor_SMD:R_0805_2012Metric_Pad1.20x1.40mm_HandSolder" (id 2) (at 46.99 142.748 90)
+    (property "Footprint" "Resistor_SMD:R_0603_1608Metric_Pad0.98x0.95mm_HandSolder" (id 2) (at 46.99 142.748 90)
       (effects (font (size 1.27 1.27)) hide)
     )
@@
       (effects (font (size 1.27 1.27)) hide)
     )
-    (property "Supplier Part URL" "https://www.digikey.cz/en/products/detail/yageo/RC0805FR-071KL/727444" (id 5) (at 46.99 140.97 0)
+    (property "Supplier Part URL" "" (id 5) (at 46.99 140.97 0)
       (effects (font (size 1.27 1.27)) hide)
     )
@@
       (effects (font (size 1.27 1.27)))
     )
-    (property "Footprint" "Resistor_SMD:R_0805_2012Metric_Pad1.20x1.40mm_HandSolder" (id 2) (at 77.47 170.688 90)
+    (property "Footprint" "Resistor_SMD:R_0603_1608Metric_Pad0.98x0.95mm_HandSolder" (id 2) (at 77.47 170.688 90)
       (effects (font (size 1.27 1.27)) hide)
     )
@@
       (effects (font (size 1.27 1.27)) hide)
     )
-    (property "Supplier Part URL" "https://www.digikey.cz/en/products/detail/yageo/RC0805FR-07100RL/727543" (id 5) (at 77.47 168.91 0)
+    (property "Supplier Part URL" "" (id 5) (at 77.47 168.91 0)
       (effects (font (size 1.27 1.27)) hide)
     )
@@
       (effects (font (size 1.27 1.27)))
     )
-    (property "Footprint" "Resistor_SMD:R_0805_2012Metric_Pad1.20x1.40mm_HandSolder" (id 2) (at 224.79 99.568 90)
+    (property "Footprint" "Resistor_SMD:R_0603_1608Metric_Pad0.98x0.95mm_HandSolder" (id 2) (at 224.79 99.568 90)
       (effects (font (size 1.27 1.27)) hide)
     )
@@
       (effects (font (size 1.27 1.27)) hide)
     )
-    (property "Supplier Part URL" "https://www.digikey.cz/en/products/detail/yageo/RC0805FR-071KL/727444" (id 5) (at 224.79 97.79 0)
+    (property "Supplier Part URL" "" (id 5) (at 224.79 97.79 0)
       (effects (font (size 1.27 1.27)) hide)
     )
@@
       (effects (font (size 1.27 1.27)))
     )
-    (property "Footprint" "Resistor_SMD:R_0805_2012Metric_Pad1.20x1.40mm_HandSolder" (id 2) (at 250.19 99.568 90)
+    (property "Footprint" "Resistor_SMD:R_0603_1608Metric_Pad0.98x0.95mm_HandSolder" (id 2) (at 250.19 99.568 90)
       (effects (font (size 1.27 1.27)) hide)
     )
@@
       (effects (font (size 1.27 1.27)) hide)
     )
-    (property "Supplier Part URL" "https://www.digikey.cz/en/products/detail/yageo/RC0805FR-071KL/727444" (id 5) (at 250.19 97.79 0)
+    (property "Supplier Part URL" "" (id 5) (at 250.19 97.79 0)
       (effects (font (size 1.27 1.27)) hide)
     )
@@
       (effects (font (size 1.27 1.27)))
     )
-    (property "Footprint" "Resistor_SMD:R_0805_2012Metric_Pad1.20x1.40mm_HandSolder" (id 2) (at 46.99 147.828 90)
+    (property "Footprint" "Resistor_SMD:R_0603_1608Metric_Pad0.98x0.95mm_HandSolder" (id 2) (at 46.99 147.828 90)
       (effects (font (size 1.27 1.27)) hide)
     )
@@
       (effects (font (size 1.27 1.27)) hide)
     )
-    (property "Supplier Part URL" "https://www.digikey.cz/en/products/detail/yageo/RC0805FR-071KL/727444" (id 5) (at 46.99 146.05 0)
+    (property "Supplier Part URL" "" (id 5) (at 46.99 146.05 0)
       (effects (font (size 1.27 1.27)) hide)
     )
@@
       (effects (font (size 1.27 1.27)) (justify left))
     )
-    (property "Footprint" "Resistor_SMD:R_0805_2012Metric_Pad1.20x1.40mm_HandSolder" (id 2) (at 216.662 102.87 90)
+    (property "Footprint" "Resistor_SMD:R_0603_1608Metric_Pad0.98x0.95mm_HandSolder" (id 2) (at 216.662 102.87 90)
       (effects (font (size 1.27 1.27)) hide)
     )
@@
       (effects (font (size 1.27 1.27)) hide)
     )
-    (property "Supplier Part URL" "https://www.digikey.cz/en/products/detail/yageo/RC0805FR-072KL/727664" (id 6) (at 218.44 102.87 0)
+    (property "Supplier Part URL" "" (id 6) (at 218.44 102.87 0)
       (effects (font (size 1.27 1.27)) hide)
     )
@@
       (effects (font (size 1.27 1.27)))
     )
-    (property "Footprint" "Resistor_SMD:R_0805_2012Metric_Pad1.20x1.40mm_HandSolder" (id 2) (at 100.33 147.828 90)
+    (property "Footprint" "Resistor_SMD:R_0603_1608Metric_Pad0.98x0.95mm_HandSolder" (id 2) (at 100.33 147.828 90)
       (effects (font (size 1.27 1.27)) hide)
     )
@@
       (effects (font (size 1.27 1.27)) hide)
     )
-    (property "Supplier Part URL" "https://www.digikey.cz/en/products/detail/yageo/RC0805FR-071KL/727444" (id 5) (at 100.33 146.05 0)
+    (property "Supplier Part URL" "" (id 5) (at 100.33 146.05 0)
       (effects (font (size 1.27 1.27)) hide)
     )
@@
       (effects (font (size 1.27 1.27)) (justify right))
     )
-    (property "Footprint" "Capacitor_SMD:C_0805_2012Metric_Pad1.18x1.45mm_HandSolder" (id 2) (at 162.8648 130.81 0)
+    (property "Footprint" "Capacitor_SMD:C_0603_1608Metric_Pad1.08x0.95mm_HandSolder" (id 2) (at 162.8648 130.81 0)
       (effects (font (size 1.27 1.27)) hide)
     )
@@
       (effects (font (size 1.27 1.27)) hide)
     )
-    (property "Supplier Part URL" "https://www.digikey.cz/en/products/detail/kemet/C0805C104M3RAC7800/2211748" (id 6) (at 163.83 134.62 0)
+    (property "Supplier Part URL" "" (id 6) (at 163.83 134.62 0)
       (effects (font (size 1.27 1.27)) hide)
     )
@@
       (effects (font (size 1.27 1.27)))
     )
-    (property "Footprint" "Resistor_SMD:R_0805_2012Metric_Pad1.20x1.40mm_HandSolder" (id 2) (at 237.49 99.568 90)
+    (property "Footprint" "Resistor_SMD:R_0603_1608Metric_Pad0.98x0.95mm_HandSolder" (id 2) (at 237.49 99.568 90)
       (effects (font (size 1.27 1.27)) hide)
     )
@@
       (effects (font (size 1.27 1.27)) hide)
     )
-    (property "Supplier Part URL" "https://www.digikey.cz/en/products/detail/yageo/RC0805FR-071KL/727444" (id 5) (at 237.49 97.79 0)
-      (effects (font (size 1.27 1.27)) hide)
-    )
+    (property "Supplier Part URL" "" (id 5) (at 237.49 97.79 0)
+      (effects (font (size 1.27 1.27)) hide)
+    )

Commit message: SPI conflict solved
Parts:
- C22: footprint Capacitor_SMD:C_0805_2012Metric_Pad1.18x1.45mm_HandSolder -> Capacitor_SMD:C_0603_1608Metric_Pad1.08x0.95mm_HandSolder; Supplier Part URL https://www.digikey.cz/en/products/detail/kemet/C0805C103K5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 -> (none)
Changed lines of the file:
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@@
       (effects (font (size 1.27 1.27)) (justify left))
     )
-    (property "Footprint" "Capacitor_SMD:C_0805_2012Metric_Pad1.18x1.45mm_HandSolder" (id 2) (at 88.5952 180.34 0)
+    (property "Footprint" "Capacitor_SMD:C_0603_1608Metric_Pad1.08x0.95mm_HandSolder" (id 2) (at 88.5952 180.34 0)
       (effects (font (size 1.27 1.27)) hide)
     )
@@
       (effects (font (size 1.27 1.27)) hide)
     )
-    (property "Supplier Part URL" "https://www.digikey.cz/en/products/detail/kemet/C0805C103K5RAC7210/3317006" (id 6) (at 87.63 176.53 0)
+    (property "Supplier Part URL" "" (id 6) (at 87.63 176.53 0)
       (effects (font (size 1.27 1.27)) hide)
     )

Commit message: changed footprints for resistor arrays
Parts:
- RN10, RN11, RN12, RN13, RN9: footprint Resistor_SMD:R_Array_Convex_4x1206 -> Resistor_SMD:R_Array_Convex_4x0603
Changed lines of the file:
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@@
       (effects (font (size 1.27 1.27)) (justify right))
     )
-    (property "Footprint" "Resistor_SMD:R_Array_Convex_4x1206" (id 2) (at 182.372 34.29 90)
+    (property "Footprint" "Resistor_SMD:R_Array_Convex_4x0603" (id 2) (at 182.372 34.29 90)
       (effects (font (size 1.27 1.27)) hide)
     )
@@
       (effects (font (size 1.27 1.27)) (justify right))
     )
-    (property "Footprint" "Resistor_SMD:R_Array_Convex_4x1206" (id 2) (at 109.982 26.67 90)
+    (property "Footprint" "Resistor_SMD:R_Array_Convex_4x0603" (id 2) (at 109.982 26.67 90)
       (effects (font (size 1.27 1.27)) hide)
     )
@@
       (effects (font (size 1.27 1.27)))
     )
-    (property "Footprint" "Resistor_SMD:R_Array_Convex_4x1206" (id 2) (at 39.37 103.632 90)
+    (property "Footprint" "Resistor_SMD:R_Array_Convex_4x0603" (id 2) (at 39.37 103.632 90)
       (effects (font (size 1.27 1.27)) hide)
     )
@@
       (effects (font (size 1.27 1.27)))
     )
-    (property "Footprint" "Resistor_SMD:R_Array_Convex_4x1206" (id 2) (at 91.44 103.632 90)
+    (property "Footprint" "Resistor_SMD:R_Array_Convex_4x0603" (id 2) (at 91.44 103.632 90)
       (effects (font (size 1.27 1.27)) hide)
     )
@@
       (effects (font (size 1.27 1.27)) (justify right))
     )
-    (property "Footprint" "Resistor_SMD:R_Array_Convex_4x1206" (id 2) (at 191.262 34.29 90)
+    (property "Footprint" "Resistor_SMD:R_Array_Convex_4x0603" (id 2) (at 191.262 34.29 90)
       (effects (font (size 1.27 1.27)) hide)
     )
@@
       (effects (font (size 1.27 1.27)) (justify right))
     )
-    (property "Footprint" "Resistor_SMD:R_Array_Convex_4x1206" (id 2) (at 47.752 54.61 90)
+    (property "Footprint" "Resistor_SMD:R_Array_Convex_4x0603" (id 2) (at 47.752 54.61 90)
       (effects (font (size 1.27 1.27)) hide)
     )
@@
       (effects (font (size 1.27 1.27)) (justify right))
     )
-    (property "Footprint" "Resistor_SMD:R_Array_Convex_4x1206" (id 2) (at 233.172 92.71 90)
+    (property "Footprint" "Resistor_SMD:R_Array_Convex_4x0603" (id 2) (at 233.172 92.71 90)
       (effects (font (size 1.27 1.27)) hide)
     )
@@
       (effects (font (size 1.27 1.27)) (justify right))
     )
-    (property "Footprint" "Resistor_SMD:R_Array_Convex_4x1206" (id 2) (at 245.872 92.71 90)
+    (property "Footprint" "Resistor_SMD:R_Array_Convex_4x0603" (id 2) (at 245.872 92.71 90)
       (effects (font (size 1.27 1.27)) hide)
     )
@@
       (effects (font (size 1.27 1.27)) (justify right))
     )
-    (property "Footprint" "Resistor_SMD:R_Array_Convex_4x1206" (id 2) (at 258.572 92.71 90)
+    (property "Footprint" "Resistor_SMD:R_Array_Convex_4x0603" (id 2) (at 258.572 92.71 90)
       (effects (font (size 1.27 1.27)) hide)
     )
@@
       (effects (font (size 1.27 1.27)))
     )
-    (property "Footprint" "Resistor_SMD:R_Array_Convex_4x1206" (id 2) (at 91.44 50.292 90)
+    (property "Footprint" "Resistor_SMD:R_Array_Convex_4x0603" (id 2) (at 91.44 50.292 90)
       (effects (font (size 1.27 1.27)) hide)
     )
@@
       (effects (font (size 1.27 1.27)) (justify right))
     )
-    (property "Footprint" "Resistor_SMD:R_Array_Convex_4x1206" (id 2) (at 99.822 107.95 90)
+    (property "Footprint" "Resistor_SMD:R_Array_Convex_4x0603" (id 2) (at 99.822 107.95 90)
       (effects (font (size 1.27 1.27)) hide)
     )
@@
       (effects (font (size 1.27 1.27)) (justify right))
     )
-    (property "Footprint" "Resistor_SMD:R_Array_Convex_4x1206" (id 2) (at 109.982 80.01 90)
+    (property "Footprint" "Resistor_SMD:R_Array_Convex_4x0603" (id 2) (at 109.982 80.01 90)
       (effects (font (size 1.27 1.27)) hide)
     )
@@
       (effects (font (size 1.27 1.27)) (justify right))
     )
-    (property "Footprint" "Resistor_SMD:R_Array_Convex_4x1206" (id 2) (at 220.472 92.71 90)
+    (property "Footprint" "Resistor_SMD:R_Array_Convex_4x0603" (id 2) (at 220.472 92.71 90)
       (effects (font (size 1.27 1.27)) hide)
     )
@@
       (effects (font (size 1.27 1.27)) (justify right))
     )
-    (property "Footprint" "Resistor_SMD:R_Array_Convex_4x1206" (id 2) (at 173.482 34.29 90)
+    (property "Footprint" "Resistor_SMD:R_Array_Convex_4x0603" (id 2) (at 173.482 34.29 90)
       (effects (font (size 1.27 1.27)) hide)
     )
@@
       (effects (font (size 1.27 1.27)) (justify right))
     )
-    (property "Footprint" "Resistor_SMD:R_Array_Convex_4x1206" (id 2) (at 99.822 54.61 90)
+    (property "Footprint" "Resistor_SMD:R_Array_Convex_4x0603" (id 2) (at 99.822 54.61 90)
       (effects (font (size 1.27 1.27)) hide)
     )
@@
       (effects (font (size 1.27 1.27)) (justify right))
     )
-    (property "Footprint" "Resistor_SMD:R_Array_Convex_4x1206" (id 2) (at 47.752 107.95 90)
+    (property "Footprint" "Resistor_SMD:R_Array_Convex_4x0603" (id 2) (at 47.752 107.95 90)
       (effects (font (size 1.27 1.27)) hide)
     )
@@
       (effects (font (size 1.27 1.27)))
     )
-    (property "Footprint" "Resistor_SMD:R_Array_Convex_4x1206" (id 2) (at 39.37 50.292 90)
+    (property "Footprint" "Resistor_SMD:R_Array_Convex_4x0603" (id 2) (at 39.37 50.292 90)
       (effects (font (size 1.27 1.27)) hide)
     )
@@
       (effects (font (size 1.27 1.27)) (justify right))
     )
-    (property "Footprint" "Resistor_SMD:R_Array_Convex_4x1206" (id 2) (at 57.912 80.01 90)
+    (property "Footprint" "Resistor_SMD:R_Array_Convex_4x0603" (id 2) (at 57.912 80.01 90)
       (effects (font (size 1.27 1.27)) hide)
     )
@@
       (effects (font (size 1.27 1.27)) (justify right))
     )
-    (property "Footprint" "Resistor_SMD:R_Array_Convex_4x1206" (id 2) (at 57.912 26.67 90)
+    (property "Footprint" "Resistor_SMD:R_Array_Convex_4x0603" (id 2) (at 57.912 26.67 90)
       (effects (font (size 1.27 1.27)) hide)
     )
@@
       (effects (font (size 1.27 1.27)) (justify right))
     )
-    (property "Footprint" "Resistor_SMD:R_Array_Convex_4x1206" (id 2) (at 164.592 34.29 90)
-      (effects (font (size 1.27 1.27)) hide)
-    )
+    (property "Footprint" "Resistor_SMD:R_Array_Convex_4x0603" (id 2) (at 164.592 34.29 90)
+      (effects (font (size 1.27 1.27)) hide)
+    )
